File: Old_Repo_Dump/Antares_Raw/Double_sided/Antares_Raw_DS.kicad_pcb (KiCad board)
At the start: 6 copper layers, 83.3 x 49.5 mm, 89 parts, among them J1 USB_C_Receptacle, J2 Conn_02x05_Odd_Even, J3 Conn_01x03_Male, J4 Conn_01x01_Male, J5 Conn_01x02_Male, SW1 SW_Push, SW2 SW_Push, SW3 SW_Push, SW4 SW_SPDT, U1 BQ24073RGT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

Commit message: cleanup
Parts:
- moved FILT2 53.1 mm to (220.9, 64.2), turned to 45 degrees
- moved U7 52.4 mm to (224.3, 59.2)
- moved U5 50.8 mm to (217.7, 65.8), turned to 180 degrees
- moved C30 49.8 mm to (218.9, 62.9), turned to 135 degrees
- moved U6 47.3 mm to (211.2, 59.2), turned to 45 degrees
- moved C28 46.9 mm to (216.4, 62.9), turned to 45 degrees
- moved FILT1 45.6 mm to (214.4, 64.2), turned to 135 degrees
- moved J1 39.7 mm to (211.5, 97.0), turned to 180 degrees
- moved L1 1.46 mm to (214.8, 66.3), turned to 135 degrees
- moved Y3 1.00 mm to (213.0, 67.0)
Other:
- board size 83.3 x 49.5 mm -> 25.6 x 44.8 mm
